Commit message: add support

File: urdf/vlp16.urdf.xacro (robot description, xacro)
@@ -4,5 +4,6 @@
  <!-- <vlp16 gpu="false"/> -->
   <VLP-16 parent="top_plate_link" name="velodyne" topic="/velodyne_points" hz="10" samples="440">
-    <origin xyz="0.2206 0.0 0.00635" rpy="0 0 0" />
+    <!-- <origin xyz="0.2206 0.0 0.00635" rpy="0 0 0" /> -->
+    <origin xyz="0.2206 0.0 2.0" rpy="0 0 0" />
   </VLP-16>
 </robot>

File: urdf/vlp16_vertical.urdf.xacro (robot description, xacro)
@@ -4,5 +4,6 @@
  <!-- <vlp16 gpu="false"/> -->
   <VLP-16 parent="top_plate_link" name="velodyne" topic="/velodyne_points" hz="10" samples="440">
-    <origin xyz="0.2206 0.0 0.3" rpy="1.57 0 0" />
+    <!-- <origin xyz="0.2206 0.0 0.3" rpy="1.57 0 0" /> -->
+    <origin xyz="0.2206 0.0 2.0" rpy="1.57 0 0" />
   </VLP-16>
 </robot>
