Commit message: add filters and fixes

File: urdf/vlp16_bumblebee_vertical.urdf.xacro (robot description, xacro)
@@ -18,4 +18,8 @@
       <material name="black"/>
     </visual>
+    <!-- <inertial>
+      <mass value="0" />
+      <inertia ixx="0.0" ixy="0.0" ixz="0.0" iyy="0.0" iyz="0.0" izz="0.0" />
+    </inertial> -->
   </link>
   <joint name="base_to_support" type="fixed">
